File: buck and boost converter rev 2.kicad_sch (KiCad schematic)
At the start: 8 parts

Commit message: BOOST AND BUCK REV 3
Parts:
- added CBST, Cinx2: 100nF, Capacitor_THT:C_Disc_D3.0mm_W1.6mm_P2.50mm, symbol Device:C
- added Ccomp: 39nF, Capacitor_THT:C_Disc_D3.0mm_W1.6mm_P2.50mm, symbol Device:C
- added Ccomp2: 68nF, Capacitor_THT:C_Disc_D3.0mm_W1.6mm_P2.50mm, symbol Device:C
- added Cin2: 10uF, Capacitor_THT:C_Disc_D3.0mm_W1.6mm_P2.50mm, symbol Device:C
- added Cout2: 47uF, Capacitor_THT:C_Disc_D3.0mm_W1.6mm_P2.50mm, symbol Device:C
- added Cvcc: 2.2uF, Capacitor_THT:C_Disc_D3.0mm_W1.6mm_P2.50mm, symbol Device:C
- added L1: 4.7uH, symbol Device:L
- added Rcomp: 26.7kOhms, symbol Device:R_US
- added Rfbb: 48.7kOhms, symbol Device:R_US
- added Rfbt: 931kOhms, symbol Device:R_US
- added U2: ~, symbol 2_Converter_DCDC:TPS61288RQQ
- added V2: 1, symbol Simulation_SPICE:VDC
- Cen: footprint (none) -> Capacitor_THT:C_Disc_D3.0mm_W1.6mm_P2.50mm
- renumbered Cin to Cin1, Cinx to Cinx1, Cout to Cout1
Connections:
- net GND: now reaches Cen.2, Cin1.2, Cinx1.2, Cout1.2, R2.2, U1.4 (PGND), V1.2
- net GND: now also Ccomp.2, Ccomp2.2, Cin2.2, Cinx2.2, Cout2.2, Cvcc.2, Rfbb.2, U2.10 (AGND), U2.3 (PGND), V2.2
- new net: Ccomp.1, Rcomp.2
- new net: Cvcc.1, U2.11 (VCC)
- new net: Ccomp2.1, Rcomp.1, U2.2 (COMP)
- new net: Rfbb.1, Rfbt.2, U2.1 (FB)
- new net: Cin2.1, Cinx2.1, L1.1, U2.6 (EN), U2.7 (VIN), V2.1
- new net: CBST.1, L1.2, U2.4 (SW), U2.9 (SW)
- new net: Cout2.1, Rfbt.1, U2.5 (VOUT)
- new net: CBST.2, U2.8 (BST)
- no-connect marks 0 -> 1
Other:
- note added: "BOOST CONVERTER 4.5 V - 12V"
- moved on the sheet: Cen, Cin1, Cinx1, Cout1, R1, R2, U1, V1
